File: hardware/integrated_1/integrated_1.kicad_pcb (KiCad board)
At the start: 4 copper layers, 40 x 100 mm, 118 parts, among them J1 USB4105-GF-A-120, J2 HDMI_A_1.4, J3 DEBUG, SW1 DNF, SW2 DNF, SW3 DNF, U1 XC6SLX9-TQG144, U2 IS25LP128F-JBLE-TR, U3 W25Q16JV, U4 RP2040, U5 FT24C04A, U6 AP5725, U7 TPS650250RHBR, Y1 12MHz

Commit message: finalizing the schematic and layout
Parts:
- removed JP1, JP2, JP3, JP4: SolderJumper_2_Open, Jumper:SolderJumper-2_P1.3mm_Open_RoundedPad1.0x1.5mm
- added C54: 10n, KiCAD Library:C_0402_1005Metric, F.Cu at (187.5, 85.3)
- added G***: LOGO, LOGO, F.Cu at (176.4, 52.0)
- added J4: Conn_01x12, Connector_PinHeader_1.00mm:PinHeader_2x06_P1.00mm_Vertical_SMD, F.Cu at (188.5, 100.0)
- added REF**: OSHW-Symbol_6.7x6mm_SilkScreen, Symbol:OSHW-Symbol_6.7x6mm_SilkScreen, F.Cu at (190.4, 46.5)
- added REF**: ESD-Logo_6.6x6mm_SilkScreen, Symbol:ESD-Logo_6.6x6mm_SilkScreen, F.Cu at (189.7, 78.2)
- added U8: XLH335200.000000I, KiCAD Library:XLH335200.000000I, F.Cu at (189.8, 83.5)
- moved C24 45.7 mm to (188.6, 50.7), turned to 0 degrees
- moved U2 43.6 mm to (190.0, 56.0), turned to 90 degrees
- moved JP5 9.91 mm to (188.6, 94.6)
- moved JP6 9.91 mm to (188.6, 92.1)
- moved JP7 9.91 mm to (188.6, 89.6)
- moved JP8 9.91 mm to (188.6, 87.1)
- moved C13 0.96 mm to (186.7, 81.5), turned to 0 degrees
- moved C7 0.68 mm to (186.7, 84.6), turned to 0 degrees
- moved G*** 0.66 mm to (189.7, 110.6)
- moved C20 0.47 mm to (161.2, 80.2)
Connections:
- C13 pad 1: /FPGA IO Bank A/FPGA_{BANK0} -> +3V3
- C14 pad 1: /FPGA IO Bank A/FPGA_{BANK0} -> +3V3
- C15 pad 1: /FPGA IO Bank A/FPGA_{BANK0} -> +3V3
- C16 pad 1: /FPGA IO Bank A/FPGA_{BANK1} -> +3V3
- C17 pad 1: /FPGA IO Bank A/FPGA_{BANK1} -> +3V3
- C18 pad 1: /FPGA IO Bank A/FPGA_{BANK1} -> +3V3
- U1 pad 103: /FPGA IO Bank A/FPGA_{BANK1} -> +3V3
- U1 pad 111: unconnected-(U1A-IO_L66N_SCP0_0-Pad111) -> /FPGA IO Bank A/PMOD_A7
- U1 pad 112: unconnected-(U1A-IO_L66P_SCP1_0-Pad112) -> /FPGA IO Bank A/PMOD_A6
- U1 pad 114: unconnected-(U1A-IO_L65N_SCP2_0-Pad114) -> /FPGA IO Bank A/PMOD_A5
- U1 pad 115: unconnected-(U1A-IO_L65P_SCP3_0-Pad115) -> /FPGA IO Bank A/PMOD_A4
- U1 pad 116: unconnected-(U1A-IO_L64N_SCP4_0-Pad116) -> /FPGA IO Bank A/PMOD_A3
- U1 pad 117: unconnected-(U1A-IO_L64P_SCP5_0-Pad117) -> /FPGA IO Bank A/PMOD_A2
- U1 pad 118: unconnected-(U1A-IO_L63N_SCP6_0-Pad118) -> /FPGA IO Bank A/PMOD_A1
- U1 pad 119: unconnected-(U1A-IO_L63P_SCP7_0-Pad119) -> /FPGA IO Bank A/PMOD_A0
- U1 pad 122: /FPGA IO Bank A/FPGA_{BANK0} -> +3V3
- U1 pad 125: /FPGA IO Bank A/FPGA_{BANK0} -> +3V3
- U1 pad 133: unconnected-(U1A-IO_L34N_GCLK18_0-Pad133) -> /FPGA IO Bank A/CLK_{100N}
- U1 pad 134: unconnected-(U1A-IO_L34P_GCLK19_0-Pad134) -> /FPGA IO Bank A/CLK_{100P}
- U1 pad 135: /FPGA IO Bank A/FPGA_{BANK0} -> +3V3
- U1 pad 38: /FPGA IO Bank B/LED7 -> /FPGA IO Bank B/~{CS}
- U1 pad 39: /FPGA IO Bank B/LED6 -> /FPGA IO Bank B/LED7
- U1 pad 40: /FPGA IO Bank B/LED5 -> /FPGA IO Bank B/LED6
- U1 pad 41: /FPGA IO Bank B/LED4 -> /FPGA IO Bank B/LED5
- U1 pad 43: /FPGA IO Bank B/LED3 -> /FPGA IO Bank B/LED4
- U1 pad 44: /FPGA IO Bank B/LED2 -> /FPGA IO Bank B/LED3
- U1 pad 45: /FPGA IO Bank B/LED1 -> /FPGA IO Bank B/LED2
- U1 pad 46: /FPGA IO Bank B/LED0 -> /FPGA IO Bank B/LED1
- U1 pad 47: unconnected-(U1B-IO_L48N_RDWR_B_VREF_2-Pad47) -> /FPGA IO Bank B/LED0
- U1 pad 61: unconnected-(U1B-IO_L12N_D2_MISO3_2-Pad61) -> /FPGA IO Bank B/D_{3}
- U1 pad 62: unconnected-(U1B-IO_L12P_D1_MISO2_2-Pad62) -> /FPGA IO Bank B/D_{2}
- U1 pad 64: unconnected-(U1B-IO_L3N_MOSI_CSI_B_MISO0_2-Pad64) -> /FPGA IO Bank B/D_{0}
- U1 pad 65: unconnected-(U1B-IO_L3P_D0_DIN_MISO_MISO1_2-Pad65) -> /FPGA IO Bank B/D_{1}
- U1 pad 70: unconnected-(U1B-IO_L1P_CCLK_2-Pad70) -> /FPGA IO Bank B/CLK
- U1 pad 71: unconnected-(U1C-DONE_2-Pad71) -> /DONE
- U1 pad 76: /FPGA IO Bank A/FPGA_{BANK1} -> +3V3
- U1 pad 86: /FPGA IO Bank A/FPGA_{BANK1} -> +3V3
- U2 pad 1: unconnected-(U2-~{CE}-Pad1) -> /FPGA IO Bank B/~{CS}
- U2 pad 2: unconnected-(U2-SO-Pad2) -> /FPGA IO Bank B/D_{1}
- U2 pad 3: unconnected-(U2-~{WP}-Pad3) -> /FPGA IO Bank B/D_{2}
- U2 pad 5: unconnected-(U2-SI-Pad5) -> /FPGA IO Bank B/D_{0}
- U2 pad 6: unconnected-(U2-SCK-Pad6) -> /FPGA IO Bank B/CLK
- U2 pad 7: unconnected-(U2-~{HOLD}-Pad7) -> /FPGA IO Bank B/D_{3}
- U3 pad 9: (no net) -> GND
- U4 pad 31: unconnected-(U4-GPIO20-Pad31) -> /DONE
Routing:
- net /FPGA IO Bank B/CLK: track 0.00 -> 63.3 mm, vias 0 -> 2
- net /FPGA IO Bank B/D_{0}: track 0.00 -> 59.9 mm, vias 0 -> 2
- net +3V3: track 50.0 -> 109.1 mm, vias 22 -> 28
- net /FPGA IO Bank B/D_{2}: track 0.00 -> 58.4 mm, vias 0 -> 2
- net /FPGA IO Bank B/D_{1}: track 0.00 -> 57.3 mm, vias 0 -> 2
- net /FPGA IO Bank B/~{CS}: track 0.00 -> 55.7 mm, vias 0 -> 2
- net /FPGA IO Bank B/D_{3}: track 0.00 -> 55.5 mm, vias 0 -> 2
- net /FPGA IO Bank B/FPGA_{BANK2}: track 5.69 -> 40.4 mm
- net /FPGA IO Bank B/FPGA_{BANK3}: track 14.0 -> 46.6 mm
- net /FPGA IO Bank A/PMOD_A1: track 0.00 -> 30.4 mm, vias 0 -> 2
- net /FPGA IO Bank A/FPGA_{BANK1}: track 29.9 -> 0.00 mm, vias 4 -> 0
- net /FPGA IO Bank A/PMOD_A3: track 0.00 -> 25.9 mm, vias 0 -> 2
- net /FPGA IO Bank A/PMOD_A5: track 0.00 -> 21.1 mm, vias 0 -> 2
- net /DONE: track 0.00 -> 14.7 mm, vias 0 -> 2
- net /FPGA IO Bank A/PMOD_A7: track 0.00 -> 14.0 mm, vias 0 -> 2
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- removed copper zone on B.Cu, net /FPGA IO Bank A/FPGA_{BANK0}
- removed copper zone on B.Cu, net /FPGA IO Bank A/FPGA_{BANK1}
- removed copper zone on B.Cu, net /FPGA IO Bank B/FPGA_{BANK2}
- removed copper zone on B.Cu, net /FPGA IO Bank B/FPGA_{BANK3}
Other:
- board text added: "μPMOD"
- board text removed: "V_{CCO_{0}}"
- board text removed: "V_{CCO_{1}}"

Commit message: added testpoints
Parts:
- removed REF**: OSHW-Symbol_6.7x6mm_SilkScreen, Symbol:OSHW-Symbol_6.7x6mm_SilkScreen
- removed REF**: ESD-Logo_6.6x6mm_SilkScreen, Symbol:ESD-Logo_6.6x6mm_SilkScreen
- added J5: DNM, Connector_PinHeader_1.00mm:PinHeader_2x06_P1.00mm_Vertical_SMD, B.Cu at (168.9, 98.4)
- added TP1: TestPoint, TestPoint:TestPoint_Pad_D1.0mm, B.Cu at (180.0, 96.8)
- added TP10: TestPoint, TestPoint:TestPoint_Pad_D1.0mm, B.Cu at (191.3, 131.5)
- added TP11: TestPoint, TestPoint:TestPoint_Pad_D1.0mm, B.Cu at (189.8, 138.9)
- added TP12: TestPoint, TestPoint:TestPoint_Pad_D1.0mm, B.Cu at (176.5, 135.4)
- added TP2: TestPoint, TestPoint:TestPoint_Pad_D1.0mm, B.Cu at (170.5, 88.0)
- added TP3: TestPoint, TestPoint:TestPoint_Pad_D1.0mm, B.Cu at (163.2, 92.2)
- added TP4: TestPoint, TestPoint:TestPoint_Pad_D1.0mm, B.Cu at (163.2, 87.8)
- added TP5: TestPoint, TestPoint:TestPoint_Pad_D1.0mm, B.Cu at (176.8, 86.8)
- added TP6: TestPoint, TestPoint:TestPoint_Pad_D1.0mm, B.Cu at (185.5, 66.2)
- added TP7: TestPoint, TestPoint:TestPoint_Pad_D1.0mm, B.Cu at (182.6, 69.6)
- added TP8: TestPoint, TestPoint:TestPoint_Pad_D1.0mm, B.Cu at (170.4, 137.9)
- added TP9: TestPoint, TestPoint:TestPoint_Pad_D1.0mm, B.Cu at (186.4, 120.5)
- moved G*** 0.95 mm to (189.7, 111.6)
Routing:
- net /RP2040/SWD: track 64.2 -> 48.0 mm
- net /RP2040/SWCLK: track 59.7 -> 45.5 mm
- net GND: track 47.0 -> 57.1 mm, vias 62 -> 67
- net +3V3: track 109.1 -> 117.6 mm
- net /VCC_{AUX}: track 23.6 -> 29.6 mm
- net /TDI: track 37.8 -> 43.5 mm
- net /TCK: track 36.0 -> 40.2 mm, vias 2 -> 4
- net /TDO: track 36.6 -> 40.3 mm, vias 2 -> 4
- net /LEDA: track 0.00 -> 2.54 mm, vias 0 -> 1
- net /FPGA_D6: track 6.38 -> 8.79 mm, vias 0 -> 1
- net /FPGA_WR: track 15.3 -> 17.7 mm, vias 0 -> 1
- net +2V5: track 0.00 -> 2.39 mm
- net /FPGA_D0: track 13.2 -> 15.2 mm, vias 0 -> 1
- net /FPGA_D5: track 7.60 -> 9.61 mm, vias 0 -> 1
- net /FPGA_D1: track 12.5 -> 14.5 mm, vias 0 -> 1
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Other:
- board text added: "DATABUS"
- board text added: "GND"
- board text added: "LED"
- board text added: "TCK"
- board text added: "TDI"
- board text added: "TDO"
- board text added: "TMS"
- board text added: "V_{2V5}"
- board text added: "V_{3V3}"
- board text added: "V_{AUX}"
- board text added: "V_{INT}"

Commit message: exported 3d models + added date stamp
Parts:
- added TP13: TestPoint, TestPoint:TestPoint_Pad_D1.0mm, B.Cu at (180.0, 135.4)
- added TP14: TestPoint, TestPoint:TestPoint_Pad_D1.0mm, B.Cu at (182.2, 124.9)
- R12: footprint KiCAD Library:R_0402_1005Metric -> KiCAD Library:R_0603_1608Metric
- moved R12 1.21 mm to (183.2, 69.2)
- moved G*** 0.80 mm to (189.7, 110.8)
Routing:
- net GND: track 57.1 -> 60.0 mm, vias 67 -> 72
Other:
- board text added: "April 2024"
- board text added: "VCCO_{2}"
- board text added: "VCCO_{3}"
- board text added: "V_{5V}"
- board text removed: "V_{CCO_{2}}"
- board text removed: "V_{CCO_{3}}"
