File: hardware/integrated_1/integrated_1.kicad_pcb (KiCad board)
At the start: 4 copper layers, 40 x 100 mm, 133 parts, among them J1 USB4105-GF-A-120, J2 HDMI_A_1.4, J3 DEBUG, J4 Conn_01x12, J5 DNM, SW1 DNF, SW2 DNF, SW3 DNF, U1 XC6SLX9-TQG144, U2 IS25LP128F-JBLE-TR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

Commit message: fixed critical issue - display connector was mirrored
Parts:
- DS1: footprint KiCAD Library:GCT_FFC2B35-40-G_REVA2 -> KiCAD Library:GCT_FFC2B35-40-G_REVA2_INV
- moved SW1 36.5 mm to (190.5, 71.7)
- moved L1 34.9 mm to (157.8, 58.6), turned to 180 degrees
- moved D10 32.3 mm to (157.8, 55.5), turned to 180 degrees
- moved C41 32.0 mm to (156.7, 62.5), turned to -90 degrees
- moved U6 31.1 mm to (158.6, 63.5)
- moved R11 29.9 mm to (160.6, 62.5), turned to 90 degrees
- moved C1 29.7 mm to (187.7, 61.5), turned to 0 degrees
- moved C2 29.4 mm to (187.7, 62.4), turned to 0 degrees
- moved C42 27.6 mm to (160.9, 56.5)
- moved TP7 26.3 mm to (158.2, 60.0)
- moved R12 24.7 mm to (158.6, 66.4), turned to 180 degrees
- moved TP6 23.9 mm to (162.4, 60.0)
Connections:
- U1 pad 1: /~{RST} -> /DB17
- U1 pad 10: /HS -> /DB10
- U1 pad 11: /DB0 -> /DB9
- U1 pad 12: /DB1 -> /DB8
- U1 pad 14: /DB2 -> /DB7
- U1 pad 15: /DB3 -> /DB6
- U1 pad 16: /DB4 -> /DB5
- U1 pad 17: /DB5 -> /DB4
- U1 pad 2: /SDA -> /DB16
- U1 pad 21: /DB6 -> /DB3
- U1 pad 22: /DB7 -> /DB2
- U1 pad 23: /DB8 -> /DB1
- U1 pad 24: /DB9 -> /DB0
- U1 pad 26: /DB10 -> /HS
- U1 pad 27: /DB11 -> /VS
- U1 pad 29: /DB12 -> /DE
- U1 pad 30: /DB13 -> /DCLK
- U1 pad 32: /DB14 -> /CS
- U1 pad 33: /DB15 -> /SCL
- U1 pad 34: /DB16 -> /SDA
- U1 pad 35: /DB17 -> /~{RST}
- U1 pad 5: /SCL -> /DB15
- U1 pad 6: /CS -> /DB14
- U1 pad 7: /DCLK -> /DB13
- U1 pad 8: /DE -> /DB12
- U1 pad 9: /VS -> /DB11
Routing:
- net /BL_PWM: track 111.4 -> 83.1 mm, vias 4 -> 2
- net /TP_RST: track 48.6 -> 72.6 mm, vias 0 -> 2
- net /TP_SCL: track 48.1 -> 70.6 mm, vias 0 -> 2
- net /TP_SDA: track 47.6 -> 68.7 mm, vias 0 -> 2
- net /TP_INT: track 46.3 -> 66.1 mm, vias 0 -> 2
- net GND: track 60.0 -> 77.9 mm, vias 72 -> 76
- net /FPGA JTAG/FPGA_RST: track 24.7 -> 32.2 mm
- net /LEDA: track 2.54 -> 9.47 mm
- net +5V: track 13.7 -> 11.2 mm
- net +3V3: vias 28 -> 29
