File: hardware/integrated_1/sheets/buck_power.kicad_sch (KiCad schematic)
At the start: 29 parts, among them U5 TPS650250RHBR

Commit message: reannotated schematic
Parts:
- C39: renamed from C29; footprint Capacitor_SMD:C_0603_1608Metric -> KiCAD Library:C_0603_1608Metric
- C40: renamed from C30; footprint Capacitor_SMD:C_0603_1608Metric -> KiCAD Library:C_0402_1005Metric
- C41: renamed from C31; footprint Capacitor_SMD:C_0603_1608Metric -> KiCAD Library:C_0603_1608Metric
- C42: renamed from C32; footprint Capacitor_SMD:C_0603_1608Metric -> KiCAD Library:C_0603_1608Metric
- C43: renamed from C41; footprint Capacitor_SMD:C_0603_1608Metric -> KiCAD Library:C_0603_1608Metric
- C44: renamed from C42; footprint Capacitor_SMD:C_0603_1608Metric -> KiCAD Library:C_0603_1608Metric
- C45: renamed from C35; footprint Capacitor_SMD:C_0603_1608Metric -> KiCAD Library:C_0603_1608Metric
- C46: renamed from C36; footprint Capacitor_SMD:C_0603_1608Metric -> KiCAD Library:C_0603_1608Metric
- C47: renamed from C37; footprint Capacitor_SMD:C_0603_1608Metric -> KiCAD Library:C_0603_1608Metric
- C48: renamed from C38; footprint Capacitor_SMD:C_0603_1608Metric -> KiCAD Library:C_0603_1608Metric
- C49: renamed from C39; footprint Capacitor_SMD:C_0603_1608Metric -> KiCAD Library:C_0603_1608Metric
- C50: renamed from C40; footprint Capacitor_SMD:C_0603_1608Metric -> KiCAD Library:C_0603_1608Metric
- L2, L3, L4: footprint (none) -> KiCAD Library:XRNR4012
- R11: renamed from R10; footprint Resistor_SMD:R_0402_1005Metric -> KiCAD Library:R_0402_1005Metric
- R12: renamed from R11; footprint Resistor_SMD:R_0402_1005Metric -> KiCAD Library:R_0402_1005Metric
- R13: renamed from R12; footprint Resistor_SMD:R_0402_1005Metric -> KiCAD Library:R_0402_1005Metric
- R14: renamed from R21; footprint Resistor_SMD:R_0402_1005Metric -> KiCAD Library:R_0402_1005Metric
- R15: renamed from R22; footprint Resistor_SMD:R_0402_1005Metric -> KiCAD Library:R_0402_1005Metric
- R16: renamed from R13; footprint Resistor_SMD:R_0402_1005Metric -> KiCAD Library:R_0402_1005Metric
- R17: renamed from R14; footprint Resistor_SMD:R_0402_1005Metric -> KiCAD Library:R_0402_1005Metric
- R18: renamed from R15; footprint Resistor_SMD:R_0402_1005Metric -> KiCAD Library:R_0402_1005Metric
- R19: renamed from R16; footprint Resistor_SMD:R_0402_1005Metric -> KiCAD Library:R_0402_1005Metric
- R20: renamed from R17; footprint Resistor_SMD:R_0402_1005Metric -> KiCAD Library:R_0402_1005Metric
- R21: renamed from R18; footprint Resistor_SMD:R_0402_1005Metric -> KiCAD Library:R_0402_1005Metric
- R22: renamed from R19; footprint Resistor_SMD:R_0402_1005Metric -> KiCAD Library:R_0402_1005Metric
- R23: renamed from R20; footprint Resistor_SMD:R_0402_1005Metric -> KiCAD Library:R_0402_1005Metric
Connections:
- net VCC_{AUX}: no longer C43.1, C44.1, L2.2, R14.1, U5.8 (VDCDC1)
- net L3: now reaches L4.1, U5.3 (L3)
- net L2: now reaches L3.1, U5.27 (L2)
- net L1: now reaches L2.1, U5.6 (L1)
- new net VCC_{INT}: C43.1, C44.1, L2.2, R14.1, U5.8 (VDCDC1)
Other:
- moved on the sheet: L2, L3, L4

Commit message: reannotated
Parts:
- removed C45: 2u2, KiCAD Library:C_0603_1608Metric, symbol Device:C_Small
- removed R16, R17: 470k, KiCAD Library:R_0402_1005Metric, symbol Device:R_Small
- renumbered C39 to C43, C40 to C44, C41 to C45, C42 to C46, C43 to C47, C44 to C48, C46 to C49, C47 to C50, C48 to C51, C49 to C52, C50 to C53, R11 to R13, R12 to R14, R13 to R15, R14 to R16, R15 to R17, U5 to U7
Connections:
- net GND: now also U7.34 (EP), U7.35 (EP), U7.36 (EP), U7.37 (EP), U7.38 (EP)
- net VCC_RC: now reaches C44.1, R14.2, U7.29 (VCC)
- net FB_{DCDC_{1}}: now reaches R16.2, R17.1, U7.9 (DEFDCDC1)
- net VCC_{LDO_{2}}: no longer names the net of U7.10 (FB_LDO2)
- net VCC_{LDO_{2}}: no longer U7.14 (VLDO2)
- no-connect marks 1 -> 5
Other:
- note added: "This is completely overkill for this circuit. We could have gotten away with a significantly cheaper 3V3 and 1V2 supply with a few bucks, but this is honestly easier as we can just reference TI's existing reference design"
- note removed: "This is completely overkill for this circuit. We could have gotten away with a significantly cheaper 3V3 and 1V2 supply with a few bucks, but this is honestly cheaper as we can just reference TI's existing reference design"

Commit message: added testpoints
Parts:
- added TP10, TP11, TP12, TP8, TP9: TestPoint, TestPoint:TestPoint_Pad_D1.0mm, symbol Connector:TestPoint
Connections:
- net GND: now also TP12.1
- net VCC_{AUX}: now also TP9.1
- net VCC_{BUCK}: now also TP10.1
- net VCC_{INT}: now also TP8.1
- net VCC_{LDO_{1}}: now also TP11.1

Commit message: exported 3d models + added date stamp
Parts:
- added TP13, TP14: TestPoint, TestPoint:TestPoint_Pad_D1.0mm, symbol Connector:TestPoint
Connections:
- net GND: now also TP14.1
- net V_{IN}: now also TP13.1
Changed lines of the file:
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@@
 	)
 	(junction
+		(at 44.45 59.69)
+		(diameter 0)
+		(color 0 0 0 0)
+	)
+	(junction
 		(at 152.4 59.69)
 		(diameter 0)
@@
 	)
 	(junction
+		(at 67.31 96.52)
+		(diameter 0)
+		(color 0 0 0 0)
+	)
+	(junction
 		(at 234.95 78.74)
 		(diameter 0)
@@
 	(wire
 		(pts
-			(xy 43.18 59.69) (xy 52.07 59.69)
+			(xy 43.18 59.69) (xy 44.45 59.69)
 		)
 		(stroke
@@
 	(wire
 		(pts
+			(xy 44.45 59.69) (xy 52.07 59.69)
+		)
+		(stroke
+			(width 0)
+			(type default)
+		)
+	)
+	(wire
+		(pts
 			(xy 245.11 71.12) (xy 245.11 72.39)
 		)
@@
 	(wire
 		(pts
+			(xy 44.45 57.15) (xy 44.45 59.69)
+		)
+		(stroke
+			(width 0)
+			(type default)
+		)
+	)
+	(wire
+		(pts
 			(xy 54.61 81.28) (xy 54.61 82.55)
 		)
@@
 	(wire
 		(pts
+			(xy 67.31 92.71) (xy 67.31 96.52)
+		)
+		(stroke
+			(width 0)
+			(type default)
+		)
+	)
+	(wire
+		(pts
 			(xy 63.5 81.28) (xy 72.39 81.28)
 		)
@@
 	)
 	(symbol
+		(lib_id "Connector:TestPoint")
+		(at 44.45 57.15 0)
+		(unit 1)
+		(exclude_from_sim no)
+		(in_bom yes)
+		(on_board yes)
+		(dnp no)
+		(property "Reference" "TP13"
+			(at 42.672 51.816 0)
+			(effects
+				(font
+					(size 1.27 1.27)
+				)
+				(justify left)
+			)
+		)
+		(property "Value" "TestPoint"
+			(at 46.99 55.1179 0)
+			(effects
+				(font
+					(size 1.27 1.27)
+				)
+				(justify left)
+				(hide yes)
+			)
+		)
+		(property "Footprint" "TestPoint:TestPoint_Pad_D1.0mm"
+			(at 49.53 57.15 0)
+			(effects
+				(font
+					(size 1.27 1.27)
+				)
+				(hide yes)
+			)
+		)
+		(property "Datasheet" "~"
+			(at 49.53 57.15 0)
+			(effects
+				(font
+					(size 1.27 1.27)
+				)
+				(hide yes)
+			)
+		)
+		(property "Description" "test point"
+			(at 44.45 57.15 0)
+			(effects
+				(font
+					(size 1.27 1.27)
+				)
+				(hide yes)
+			)
+		)
+		(pin "1"
+		)
+		(instances
+			(project "integrated_1"
+				(path "/5cc60e42-d666-4a43-b4f0-3784ee4bf951/b31ef56e-e56f-49fc-b7d7-d1f43d8c5f5f"
+					(reference "TP13")
+					(unit 1)
+				)
+			)
+		)
+	)
+	(symbol
 		(lib_id "power:GND")
 		(at 245.11 80.01 0)
@@
 					(unit 1)
 				)
+			)
+		)
+	)
+	(symbol
+		(lib_id "Connector:TestPoint")
+		(at 67.31 92.71 0)
+		(unit 1)
+		(exclude_from_sim no)
+		(in_bom yes)
+		(on_board yes)
+		(dnp no)
+		(property "Reference" "TP14"
+			(at 65.532 87.376 0)
+			(effects
+				(font
+					(size 1.27 1.27)
+				)
+				(justify left)
+			)
+		)
+		(property "Value" "TestPoint"
+			(at 69.85 90.6779 0)
+			(effects
+				(font
+					(size 1.27 1.27)
+				)
+				(justify left)
+				(hide yes)
+			)
+		)
+		(property "Footprint" "TestPoint:TestPoint_Pad_D1.0mm"
+			(at 72.39 92.71 0)
+			(effects
+				(font
+					(size 1.27 1.27)
+				)
+				(hide yes)
+			)
+		)
+		(property "Datasheet" "~"
+			(at 72.39 92.71 0)
+			(effects
+				(font
+					(size 1.27 1.27)
+				)
+				(hide yes)
+			)
+		)
+		(property "Description" "test point"
+			(at 67.31 92.71 0)
+			(effects
+				(font
+					(size 1.27 1.27)
+				)
+				(hide yes)
+			)
+		)
+		(pin "1"
+		)
+		(instances
+			(project "integrated_1"
+				(path "/5cc60e42-d666-4a43-b4f0-3784ee4bf951/b31ef56e-e56f-49fc-b7d7-d1f43d8c5f5f"
+					(reference "TP14")
+					(unit 1)
+				)
