File: hardware/integrated_1/sheets/rp2040.kicad_sch (KiCad schematic)
At the start: 25 parts, among them SW1 DNF, SW2 DNF, U4 W25Q16JV, U5 RP2040, Y1 12MHz

Commit message: renaming a few pins
Connections:
- net BL_PWM: now reaches U5.4 (GPIO2)
- no-connect marks 9 -> 8
Changed lines of the file:
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@@
-	)
-	(no_connect
-		(at 173.99 76.2)
 	)
 	(no_connect
@@
 		(pts
 			(xy 173.99 129.54) (xy 176.53 129.54)
+		)
+		(stroke
+			(width 0)
+			(type default)
+		)
+	)
+	(wire
+		(pts
+			(xy 173.99 76.2) (xy 176.53 76.2)
 		)
 		(stroke
@@
 		(fields_autoplaced yes)
 		(effects
+			(font
+				(size 1.27 1.27)
+			)
+			(justify left)
+		)
+	)
+	(hierarchical_label "BL_PWM"
+		(shape output)
+		(at 176.53 76.2 0)
+		(fields_autoplaced yes)
+		(effects

Commit message: moved usb resistors inside the rp2040 sheet
Parts:
- added R6, R7: 27, Resistor_SMD:R_0402_1005Metric, symbol Device:R_Small
- R3: renamed from R9; footprint Resistor_SMD:R_0603_1608Metric -> Resistor_SMD:R_0402_1005Metric
- R4: renamed from R10; footprint Resistor_SMD:R_0603_1608Metric -> Resistor_SMD:R_0402_1005Metric
- R5: renamed from R11; footprint Resistor_SMD:R_0603_1608Metric -> Resistor_SMD:R_0402_1005Metric
- R8: renamed from R12; footprint Resistor_SMD:R_0603_1608Metric -> Resistor_SMD:R_0402_1005Metric
- renumbered C3 to C12, C4 to C13, C5 to C14, C6 to C15, C7 to C16, C8 to C17, C9 to C18, C10 to C19, C11 to C20, C12 to C21, C13 to C22, C14 to C23, C15 to C24, C16 to C25, C17 to C26, U4 to U2, U5 to U3
Connections:
- net USB_D+: now also R6.1; no longer U3.47 (USB_DP)
- net USB_D-: now also R7.1; no longer U3.46 (USB_DM)
- net PWR_CYC: now reaches U3.17 (GPIO14)
- net ~{PWR_FAIL}: now reaches U3.18 (GPIO15)
- new net D+: R6.2, U3.47 (USB_DP)
- new net D-: R7.2, U3.46 (USB_DM)
- no-connect marks 8 -> 6

Commit message: reannotated schematic
Parts:
- C22: renamed from C12; footprint Capacitor_SMD:C_0402_1005Metric -> KiCAD Library:C_0402_1005Metric
- C23: renamed from C13; footprint Capacitor_SMD:C_0402_1005Metric -> KiCAD Library:C_0402_1005Metric
- C24: renamed from C14; footprint Capacitor_SMD:C_0402_1005Metric -> KiCAD Library:C_0402_1005Metric
- C26: renamed from C16; footprint Capacitor_SMD:C_0402_1005Metric -> KiCAD Library:C_0402_1005Metric
- C27: renamed from C17; footprint Capacitor_SMD:C_0402_1005Metric -> KiCAD Library:C_0402_1005Metric
- C28: renamed from C18; footprint Capacitor_SMD:C_0402_1005Metric -> KiCAD Library:C_0402_1005Metric
- C29: renamed from C19; footprint Capacitor_SMD:C_0402_1005Metric -> KiCAD Library:C_0402_1005Metric
- C30: renamed from C20; footprint Capacitor_SMD:C_0402_1005Metric -> KiCAD Library:C_0402_1005Metric
- C31: renamed from C21; footprint Capacitor_SMD:C_0402_1005Metric -> KiCAD Library:C_0402_1005Metric
- C32: renamed from C22; footprint Capacitor_SMD:C_0402_1005Metric -> KiCAD Library:C_0402_1005Metric
- C33: renamed from C23; footprint Capacitor_SMD:C_0402_1005Metric -> KiCAD Library:C_0402_1005Metric
- C34: renamed from C24; footprint Capacitor_SMD:C_0402_1005Metric -> KiCAD Library:C_0402_1005Metric
- C35: renamed from C25; footprint Capacitor_SMD:C_0402_1005Metric -> KiCAD Library:C_0402_1005Metric
- C36: renamed from C26; footprint Capacitor_SMD:C_0402_1005Metric -> KiCAD Library:C_0402_1005Metric
- R3, R4, R5, R6, R7, R8: footprint Resistor_SMD:R_0402_1005Metric -> KiCAD Library:R_0402_1005Metric
- renumbered C15 to C25
Connections:
- net TP_INT: now also U3.32 (GPIO21); no longer U3.35 (GPIO23)
- net TP_RST: now also U3.36 (GPIO24); no longer U3.34 (GPIO22)
- net TP_SCL: now also U3.35 (GPIO23); no longer U3.32 (GPIO21)
- net TP_SDA: now also U3.34 (GPIO22); no longer U3.31 (GPIO20)

Commit message: added cheap eeprom
Parts:
- added C40: 100n, KiCAD Library:C_0402_1005Metric, symbol Device:C_Small
- added R10: 270, KiCAD Library:R_0402_1005Metric, symbol Device:R_Small
- added R9: 1k, KiCAD Library:R_0402_1005Metric, symbol Device:R_Small
- added U5: FT24C04A, Package_SO:SOIC-8_3.9x4.9mm_P1.27mm, symbol Cuprum:24C04
- D9: renamed from D1; footprint Diode_SMD:D_0805_2012Metric -> KiCAD Library:D_0805_2012Metric
- R8: value 270 -> 1k
- renumbered C22 to C25, C23 to C26, C24 to C27, C25 to C28, C26 to C29, C27 to C30, C28 to C31, C29 to C32, C30 to C33, C31 to C34, C32 to C35, C33 to C36, C34 to C37, C35 to C38, C36 to C39, SW1 to SW2, SW2 to SW3, U2 to U3, U3 to U4
Connections:
- net +3V3: now also R8.1, C40.1, R9.1, U5.8 (VCC)
- net GND: now also C40.2, U5.1 (A0), U5.2 (A1), U5.3 (A3), U5.4 (GND), U5.7 (WP)
- net LED_STATUS: now also R10.1; no longer R8.2
- net at D9.2 (A): now also R10.2; no longer R8.1
- net EEPROM_SCL: now reaches U4.40 (GPIO28_ADC2)
- net EEPROM_SCL: now also R9.2, U5.5 (SDA)
- net EEPROM_SDA: now reaches U4.41 (GPIO29_ADC3)
- net EEPROM_SDA: now also R8.2, U5.6 (SCL)
- no-connect marks 6 -> 4
Other:
- note added: "I2C ADDR: 0x50"
- moved on the sheet: D9

Commit message: finalizing the schematic and layout
Connections:
- net GND: now also U3.9 (GND)
- net DONE: now reaches U4.31 (GPIO20)
- no-connect marks 4 -> 3
Changed lines of the file:
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@@
 		(at 173.99 142.24)
 	)
-	(no_connect
-		(at 173.99 121.92)
-	)
 	(wire
 		(pts
@@
 		(pts
 			(xy 55.88 104.14) (xy 55.88 105.41)
+		)
+		(stroke
+			(width 0)
+			(type default)
+		)
+	)
+	(wire
+		(pts
+			(xy 173.99 121.92) (xy 176.53 121.92)
 		)
 		(stroke
@@
 		(shape bidirectional)
 		(at 176.53 127 0)
+		(fields_autoplaced yes)
+		(effects
+			(font
+				(size 1.27 1.27)
+			)
+			(justify left)
+		)
+	)
+	(hierarchical_label "DONE"
+		(shape input)
+		(at 176.53 121.92 0)
 		(fields_autoplaced yes)
 		(effects
@@
 		(pin "8"
 		)
+		(pin "9"
+		)
 		(instances

Commit message: exported 3d models + added date stamp
Changed lines of the file:
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@@
 	(wire
 		(pts
-			(xy 173.99 134.62) (xy 186.69 134.62)
+			(xy 173.99 134.62) (xy 187.96 134.62)
 		)
 		(stroke
@@
 	(wire
 		(pts
-			(xy 186.69 130.81) (xy 186.69 134.62)
+			(xy 187.96 130.81) (xy 187.96 134.62)
 		)
 		(stroke
@@
 	(wire
 		(pts
-			(xy 186.69 130.81) (xy 209.55 130.81)
+			(xy 187.96 130.81) (xy 209.55 130.81)
 		)
 		(stroke
@@
 	)
 	(label "LED_STATUS"
-		(at 187.96 130.81 0)
+		(at 189.23 130.81 0)
 		(fields_autoplaced yes)
 		(effects
